File: Hardware/FaultyCat.kicad_pcb (KiCad board)
At the start: 2 copper layers, 51.2 x 124.2 mm, 136 parts, among them J1 Antenna, J10 TRIGGER_VREF, J2 BG306-02-A-2-0400-L-G, J3 Conn_01x10, J4 Header 2, J5 Header 4, J6 Input Power:2x AA Battery, J7 GLITCHER_EN, J8 ANALOG_PINS, J9 TRIGGER_IN, P1 USB_C_Plug_USB2.0, Q1 AO3422, Q2 AO3422, Q3 LDA111STR, Q4 RGT16BM65DTL, Q5 DMG3415U-7, Q7 IRLML2502, Q8 IRF7807PBF, SW1 TL3305AF260QG, SW2 ON, SW3 TL3305AF260QG, SW4 RESET, SW5 BOOT, SW6 TL3305AF260QG, SW7 SW_SP3T, T1 ATB322524, T2 ATB322524, U1 AP2112K-3.3, U2 W25Q16JV, U3 RP2040, U4 TXS0108EPW, U5 TLV75718PDBV, U6 SN74LVC1T45DBV, Y1 12Mhz

Commit message: Dhiru's changes (August-2026) - WIP (hold on!)
- Port to KiCad 10.x

- Fixed ERC issues

- Fixed DRC issues

- Add a 'test suite' to catch any deviations and regressions
Parts:
- removed the G*** at (111.2, 69.5)
- J1: footprint BuggyCat:732511150 -> Connector_Coaxial:SMA_Samtec_SMA-J-P-H-ST-EM1_EdgeMount
- P1: value USB_C_Plug_USB2.0 -> USB; footprint Connectors:C393939 -> BuggyCat:USB_C_Receptacle_HRO_TYPE-C-31-M-12-Modded
- PIC1: renamed from REF**; value OSHW-Logo_7.5x8mm_SilkScreen -> OSHW_Logo
- SW2: footprint chipshouter:OS102011MA1QN1 -> BuggyCat:OS102011MA1QN1
- moved P1 3.15 mm to (110.6, 29.0)
- turned J1 to -90 degrees
- gave numbers to parts that had none: 2
- renumbered REF** to HOLE1
Connections:
- P1 pad A8: (no net) -> unconnected-(P1-SBU1-PadA8)
- P1 pad B8: (no net) -> unconnected-(P1-SBU2-PadB8)
Routing:
- net Net-(J1-Ext): track 52.9 -> 58.4 mm
- net Net-(D5-A): track 74.2 -> 69.9 mm
- net Net-(D4-K): track 36.6 -> 35.0 mm
- net +3V3: track 234.9 -> 233.6 mm
- net GND: track 167.8 -> 167.1 mm
- net Net-(J3-Pin_2): track 21.2 -> 20.6 mm
