File: Hardware/FaultyCat.kicad_sch (KiCad schematic)
At the start: 94 parts, among them J1 Antenna, J10 TRIGGER_VREF, J2 BG306-02-A-2-0400-L-G, J3 Conn_01x10, J4 Header 2, J5 Header 4, J6 Input Power:2x AA Battery, J7 GLITCHER_EN, J8 ANALOG_PINS, J9 TRIGGER_IN, P1 USB_C_Plug_USB2.0, Q1 AO3422, Q2 AO3422, Q3 LDA111STR, Q4 RGT16BM65DTL, Q5 DMG3415U-7, Q7 IRLML2502, Q8 IRF7807PBF, SW1 TL3305AF260QG, SW2 ON, SW3 TL3305AF260QG, SW4 RESET, SW5 BOOT, SW6 TL3305AF260QG, SW7 SW_SP3T, T1 ATB322524, T2 ATB322524, U1 AP2112K-3.3, U2 W25Q16JV, U3 RP2040, U4 TXS0108EPW, U5 TLV75718PDBV, U6 SN74LVC1T45DBV, Y1 12Mhz

Commit message: Dhiru's changes (August-2026) - WIP (hold on!)
- Port to KiCad 10.x

- Fixed ERC issues

- Fixed DRC issues

- Add a 'test suite' to catch any deviations and regressions
Parts:
- removed P1: USB_C_Plug_USB2.0, Connectors:C393939, symbol Connector:USB_C_Plug_USB2.0
- added P1: USB, BuggyCat:USB_C_Receptacle_HRO_TYPE-C-31-M-12-Modded, symbol usb_c_receptacle_usb2.0:USB_C_Receptacle_USB2.0
- added PIC1: OSHW_Logo, Symbol:OSHW-Logo_7.5x8mm_SilkScreen, symbol PCM_SparkFun-Aesthetic:OSHW_Logo
- J1: footprint BuggyCat:732511150 -> Connector_Coaxial:SMA_Samtec_SMA-J-P-H-ST-EM1_EdgeMount; symbol CatSniffer-rescue:Conn_Coaxial-Connector-CatStick-rescue-CatSniffer-rescue -> Connector:Conn_Coaxial
- Q5: symbol Device:Q_PMOS_GSD -> q_pmos_gsd:Q_PMOS_GSD
- Q7: symbol pico-glitcher:NMOSFETSOT23-GSD -> nmosfetsot23-gsd:NMOSFETSOT23-GSD
- Q8: symbol pico-glitcher:MOSFET-NCHANNEL-SOIC8 -> mosfet-nchannel-soic8:MOSFET-NCHANNEL-SOIC8
- SW2: footprint chipshouter:OS102011MA1QN1 -> BuggyCat:OS102011MA1QN1; now left out of the parts list
- U1: symbol HunterCat-NFC-rescue:AP2112K-3.3-Regulator_Linear -> ap2112k-3.3-regulator_linear:AP2112K-3.3-Regulator_Linear
- U3: symbol PicoWAN-rescue:RP2040-MCU_RaspberryPi_and_Boards-PicoWAN-rescue-PicoWAN-rescue -> rp2040-mcu_raspberrypi_and_boards-picowan-rescue-picowan-rescue:RP2040-MCU_RaspberryPi_and_Boards-PicoWAN-rescue-PicoWA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
Connections:
- net D+: now also P1.A6 (D+), P1.B6 (D+)
- net D-: now also P1.A7 (D-), P1.B7 (D-)
- net GND: now also P1.A1 (GND), P1.A12 (GND), P1.B1 (GND), P1.B12 (GND), P1.S1 (SHIELD)
- net at R2.1: now also P1.A5 (CC1)
- net at R4.1: now also P1.B5 (CC2)
- net at F1.1: now also P1.A4 (VBUS), P1.A9 (VBUS), P1.B4 (VBUS), P1.B9 (VBUS)
- no-connect marks 11 -> 15
Other:
- title: FaultyCat -> FaultyCat 2.2 R2
- moved on the sheet: C1, C10, C13, C14, C15, C16, C17, C18, C19, C2, C20, C3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
